File: hardware/ng-beacon.brd (EAGLE design)
At the start: 71.1 x 76.2 mm, 7 parts

Commit message: fix: change shape of boot loader pads
Parts:
- removed PAD1, PAD2: (no value), wirepad:SMD1,27-2,54
- added DFU: JUMPER-PAD-2-NO, SparkFun-Passives:PAD-JUMPER-2-NO_NO_SILK
Connections:
- net GND: now also DFU.1; no longer PAD2.1
- net N$4: now also DFU.2; no longer PAD1.1
Routing:
- net GND: track 169.4 -> 170.2 mm
Changed lines of the file:
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@@
 <attribute name="VALUE" x="44.63" y="17.735" size="0.8128" layer="27" font="vector" ratio="5" rot="R270"/>
 </element>
-<element name="PAD1" library="wirepad" package="SMD1,27-2,54" value="" x="53.975" y="13.97" smashed="yes" rot="R90">
-<attribute name="VALUE" x="53.975" y="13.97" size="0.0254" layer="27" rot="R90"/>
-</element>
-<element name="PAD2" library="wirepad" package="SMD1,27-2,54" value="" x="53.975" y="15.875" smashed="yes" rot="R90">
-<attribute name="VALUE" x="53.975" y="15.875" size="0.0254" layer="27" rot="R90"/>
+<element name="DFU" library="SparkFun-Passives" package="PAD-JUMPER-2-NO_NO_SILK" value="JUMPER-PAD-2-NO" x="53.34" y="14.605" smashed="yes" rot="R270">
+<attribute name="NAME" x="52.82" y="13.25" size="0.4064" layer="25"/>
+<attribute name="VALUE" x="51.689" y="15.513" size="0.4064" layer="27" rot="R270"/>
 </element>
 </elements>
@@
 <wire x1="41.87" y1="18.685" x2="40.005" y2="18.685" width="0.254" layer="1"/>
 <wire x1="40.005" y1="18.685" x2="40.005" y2="8.935" width="0.254" layer="1"/>
-<contactref element="PAD2" pad="1"/>
-<wire x1="53.975" y1="15.875" x2="51.435" y2="16.51" width="0.254" layer="1"/>
+<contactref element="DFU" pad="1"/>
+<wire x1="53.34" y1="15.055" x2="51.435" y2="15.055" width="0.254" layer="1"/>
+<wire x1="51.435" y1="15.055" x2="51.435" y2="16.51" width="0.254" layer="1"/>
 </signal>
 <signal name="N$1">
@@
 <signal name="N$4">
 <contactref element="U$2" pad="8"/>
-<contactref element="PAD1" pad="1"/>
+<contactref element="DFU" pad="2"/>
 <wire x1="49.72" y1="13.935" x2="53.34" y2="13.935" width="0.254" layer="1"/>
-<wire x1="53.34" y1="13.935" x2="53.975" y2="13.97" width="0.254" layer="1"/>
+<wire x1="53.34" y1="13.935" x2="53.34" y2="14.155" width="0.254" layer="1"/>
 </signal>
 </signals>
