File: hardware/ng-beacon.brd (EAGLE design)
At the start: 71.1 x 76.2 mm, 7 parts

Commit message: Convert to PTR5618, export components to project-specific library.
Parts:
- G1: device SparkFun-Electromechanical:BATTCON_20MM_4LEGS -> ng-beacon:BATTCON_20MM_4LEGS
- J3: device heathkit:PROTO4X6 -> ng-beacon:PROTO4X6
- S1: device SparkFun-Electromechanical:AYZ0202 -> ng-beacon:AYZ0202
- SN1: device sensirion:DFN6/SHT -> ng-beacon:DFN6/SHT
- U$1: value PTR5518STD -> PTR5618; device PTR5518:PTR5518 -> ng-beacon:PTR5518
Connections:
- net GND: no longer U$1.8
Routing:
- net GND: track 131.3 -> 158.6 mm
Other:
- board text added: "PO.28"
- board text removed: "PO.26"
Changed lines of the file:
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@@
 </polygon>
 <text x="74.676" y="18.542" size="1.4224" layer="25" font="fixed" rot="R83">https://github.com/urish/ng-beacon</text>
-<text x="59.69" y="41.275" size="0.6096" layer="25" rot="R90">PO.27</text>
-<text x="62.23" y="41.275" size="0.6096" layer="25" rot="R90">PO.26</text>
+<text x="59.69" y="41.275" size="0.6096" layer="25" rot="R90">PO.28</text>
+<text x="62.23" y="41.275" size="0.6096" layer="25" rot="R90">PO.27</text>
 <text x="64.77" y="41.275" size="0.6096" layer="25" rot="R90">SCL</text>
 <text x="67.31" y="41.275" size="0.6096" layer="25" rot="R90">SDA</text>
@@
 </autorouter>
 <elements>
-<element name="G1" library="SparkFun-Electromechanical" package="BATTCON_20MM_4LEGS" value="20mm coincell" x="24.13" y="51.435" rot="R270">
+<element name="G1" library="ng-beacon" package="BATTCON_20MM_4LEGS" value="20mm coincell" x="24.13" y="51.435" rot="R270">
 <attribute name="PROD_ID" value="BATT-10373" x="24.13" y="51.435" size="1.778" layer="27" rot="R270" display="off"/>
 <attribute name="VALUE" value="20mm coincell" x="24.13" y="51.435" size="1.778" layer="27" rot="R270" display="off"/>
 </element>
-<element name="U$1" library="PTR5518" package="PTR5518" value="PTR5518STD" x="45.72" y="13.97" rot="R180"/>
-<element name="S1" library="SparkFun-Electromechanical" package="AYZ0202" value="DPDT" x="71.630953125" y="60.047775" rot="R160">
+<element name="U$1" library="ng-beacon" package="PTR5518" value="PTR5618" x="45.72" y="13.97" rot="R180"/>
+<element name="S1" library="ng-beacon" package="AYZ0202" value="DPDT" x="71.630953125" y="60.047775" rot="R160">
 <attribute name="PROD_ID" value="SWCH-08179" x="71.630953125" y="60.047775" size="1.778" layer="27" rot="R160" display="off"/>
 </element>
@@
 <attribute name="VALUE" x="24.5690875" y="10.147321875" size="1.27" layer="27" rot="R329.2"/>
 </element>
-<element name="SN1" library="sensirion" package="DFN6/SHT" value="SHT21" x="71.12" y="34.29" smashed="yes">
+<element name="SN1" library="ng-beacon" package="DFN6/SHT" value="SHT21" x="71.12" y="34.29" smashed="yes">
 <attribute name="VALUE" x="73.995" y="32.415" size="0.8128" layer="27" ratio="10" rot="R90"/>
 </element>
 <element name="DFU" library="SparkFun-Passives" package="PAD-JUMPER-2-NO_NO_SILK" value="JUMPER-PAD-2-NO" x="35.56" y="13.335" rot="R270"/>
-<element name="J3" library="heathkit" package="PROTO4X6" value="" x="59.69" y="45.085" rot="R90"/>
+<element name="J3" library="ng-beacon" package="PROTO4X6" value="" x="59.69" y="45.085" rot="R90"/>
 </elements>
 <signals>
@@
 <wire x1="74.295" y1="16.51" x2="73.66" y2="15.24" width="0.254" layer="16"/>
 <contactref element="DFU" pad="2"/>
-<contactref element="U$1" pad="8"/>
 <wire x1="73.66" y1="15.24" x2="66.04" y2="11.43" width="0.254" layer="16"/>
-<wire x1="66.04" y1="11.43" x2="59.69" y2="11.43" width="0.254" layer="16"/>
+<wire x1="66.04" y1="11.43" x2="62.23" y2="11.43" width="0.254" layer="16"/>
 <via x="59.69" y="11.43" extent="1-16" drill="0.6" shape="square"/>
+<wire x1="62.23" y1="11.43" x2="59.69" y2="11.43" width="0.254" layer="16"/>
 <wire x1="59.69" y1="11.43" x2="55.88" y2="12.7" width="0.254" layer="1"/>
 <wire x1="55.88" y1="12.7" x2="52.07" y2="12.7" width="0.254" layer="1"/>
-<wire x1="39.37" y1="11.43" x2="36.83" y2="11.43" width="0.254" layer="1"/>
-<wire x1="36.83" y1="11.43" x2="35.56" y2="12.885" width="0.254" layer="1"/>
-<wire x1="36.83" y1="11.43" x2="33.76595" y2="8.213378125" width="0.254" layer="1"/>
-<wire x1="33.76595" y1="8.213378125" x2="35.56" y2="10.16" width="0.254" layer="16"/>
-<wire x1="35.56" y1="10.16" x2="27.94" y2="14.605" width="0.254" layer="16"/>
+<wire x1="33.76595" y1="8.213378125" x2="34.29" y2="10.16" width="0.254" layer="16"/>
+<wire x1="34.29" y1="10.16" x2="27.94" y2="14.605" width="0.254" layer="16"/>
 <wire x1="27.94" y1="14.605" x2="22.225" y2="14.605" width="0.254" layer="16"/>
 <wire x1="22.225" y1="14.605" x2="33.655" y2="40.005" width="0.254" layer="16"/>
@@
 <wire x1="76.68275" y1="38.046609375" x2="72.39" y2="42.339359375" width="0.254" layer="16"/>
 <wire x1="72.39" y1="42.339359375" x2="72.39" y2="45.085" width="0.254" layer="16"/>
-<wire x1="39.37" y1="11.43" x2="52.07" y2="12.7" width="0" layer="19" extent="1-1"/>
+<wire x1="62.23" y1="11.43" x2="62.23" y2="8.89" width="0.254" layer="16"/>
+<wire x1="62.23" y1="8.89" x2="56.515" y2="5.715" width="0.254" layer="16"/>
+<wire x1="56.515" y1="5.715" x2="36.195" y2="5.715" width="0.254" layer="16"/>
+<wire x1="35.56" y1="12.885" x2="33.76595" y2="8.213378125" width="0.254" layer="1"/>
+<wire x1="36.195" y1="5.715" x2="33.76595" y2="8.14405" width="0.254" layer="16"/>
+<wire x1="33.76595" y1="8.14405" x2="33.76595" y2="8.213378125" width="0.254" layer="16"/>
 </signal>
 <signal name="N$1">
