File: hardware/ng-beacon-proto.sch (EAGLE design)
At the start: 7 parts

Commit message: feat: add LED + BUTTON to the proto board
Parts:
- removed DFU: JUMPER-PAD-2-NO, SparkFun-Passives:JUMPER-PAD-2-NO
- added D1: GREEN, SparkFun-LED:LED-GREEN0603
- added R1: 470, SparkFun-Resistors:470OHM1/10W1%(0603)
- added S2: SWITCH-MOMENTARY-2SMD-1101NE, SparkFun-Electromechanical:SWITCH-MOMENTARY-2SMD-1101NE
Connections:
- new net N$7: D1.C, U$1.P0.26
- new net N$8: D1.A, R1.1
- net GND: now also S2.2; no longer DFU.2
- net N$4: now also S2.1; no longer DFU.1
- net VIN: now also R1.2
Changed lines of the file:
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@@
 <?xml version="1.0" encoding="utf-8"?>
 <!DOCTYPE eagle SYSTEM "eagle.dtd">
-<eagle version="8.0.2">
+<eagle version="7.6.0">
 <drawing>
 <settings>
@@
 <part name="SN1" library="ng-beacon" deviceset="SHT21" device=""/>
 <part name="GND4" library="SparkFun-Aesthetics" deviceset="GND" device=""/>
-<part name="DFU" library="SparkFun-Passives" deviceset="JUMPER-PAD-2-NO" device=""/>
 <part name="GND5" library="SparkFun-Aesthetics" deviceset="GND" device=""/>
 <part name="J3" library="ng-beacon" deviceset="CONN_06" device=""/>
+<part name="D1" library="SparkFun-LED" deviceset="LED-GREEN" device="0603" value="GREEN"/>
+<part name="R1" library="SparkFun-Resistors" deviceset="470OHM1/10W1%(0603)" device="" value="470"/>
+<part name="S2" library="SparkFun-Electromechanical" deviceset="SWITCH-MOMENTARY-2" device="SMD-1101NE"/>
 </parts>
 <sheets>
@@
 <instance part="SN1" gate="G$1" x="106.68" y="38.1"/>
 <instance part="GND4" gate="1" x="83.82" y="30.48" rot="R270"/>
-<instance part="DFU" gate="G$1" x="76.2" y="76.2" smashed="yes">
-<attribute name="NAME" x="71.628" y="77.47" size="1.778" layer="95"/>
-</instance>
 <instance part="GND5" gate="1" x="83.82" y="76.2" rot="R90"/>
 <instance part="J3" gate="G$1" x="7.62" y="55.88"/>
+<instance part="D1" gate="G$1" x="30.48" y="73.66" rot="R90"/>
+<instance part="R1" gate="G$1" x="22.86" y="73.66" rot="R180"/>
+<instance part="S2" gate="G$1" x="76.2" y="76.2"/>
 </instances>
 <busses>
@@
 </segment>
 <segment>
-<pinref part="DFU" gate="G$1" pin="2"/>
 <pinref part="GND5" gate="1" pin="GND"/>
+<pinref part="S2" gate="G$1" pin="2"/>
 </segment>
 </net>
@@
 <wire x1="17.78" y1="76.2" x2="17.78" y2="81.28" width="0.1524" layer="91"/>
 <label x="17.78" y="81.28" size="1.778" layer="95" rot="R90" xref="yes"/>
-<wire x1="17.78" y1="76.2" x2="17.78" y2="60.96" width="0.1524" layer="91"/>
+<wire x1="17.78" y1="76.2" x2="17.78" y2="73.66" width="0.1524" layer="91"/>
 <pinref part="J3" gate="G$1" pin="5"/>
+<wire x1="17.78" y1="73.66" x2="17.78" y2="60.96" width="0.1524" layer="91"/>
 <wire x1="12.7" y1="60.96" x2="17.78" y2="60.96" width="0.1524" layer="91"/>
+<pinref part="R1" gate="G$1" pin="2"/>
+<junction x="17.78" y="73.66"/>
 </segment>
 <segment>
@@
 </segment>
 </net>
-<net name="N$4" class="0">
-<segment>
-<pinref part="U$1" gate="G$1" pin="P0.17"/>
-<pinref part="DFU" gate="G$1" pin="1"/>
-</segment>
-</net>
 <net name="N$5" class="0">
 <segment>
@@
 </segment>
 </net>
+<net name="N$7" class="0">
+<segment>
+<pinref part="U$1" gate="G$1" pin="P0.26"/>
+<pinref part="D1" gate="G$1" pin="C"/>
+</segment>
+</net>
+<net name="N$8" class="0">
+<segment>
+<pinref part="D1" gate="G$1" pin="A"/>
+<pinref part="R1" gate="G$1" pin="1"/>
+</segment>
+</net>
+<net name="N$4" class="0">
+<segment>
+<pinref part="U$1" gate="G$1" pin="P0.17"/>
+<pinref part="S2" gate="G$1" pin="1"/>
+</segment>
+</net>
